Commit message: better tests

File: src/imetro_behavior/tests/test_data/test.urdf (robot description, URDF)
Before this commit: robot test_robot, 4 links, 3 joints
Links:
- link cylinder_link: geometry collision cylinder length=0.5 radius=0.4; visual cylinder length=0.5 radius=0.4
- link sphere_link: geometry collision sphere radius=0.6; visual sphere radius=0.6
